Commit message: go2_eskf: magnetometer heading, and fix the --adapt posture chain
Adds a magnetometer heading update to the ESKF, then fixes what the first
live terrain squares with it exposed: a sign bug that made --adapt shift
the CoM downhill, a noisy attitude estimate, a fall check and stall check
that aborted healthy runs, and magnetometer spikes leaking into yaw.

Magnetometer (use_mag, off by default until A/B'd; --mag in the launcher)
- EskfCore::correctYaw: direct psi update with a wrapped innovation.
  EskfCore::magHeading: tilt compensation from vectors (field + low-passed
  accel "up", both in the IMU frame), so the flipped sim-IMU frame is
  irrelevant. Mirrored in the NumPy twin; cross_validate.py adds a second
  stream that spins through +-pi (2.5e-15). 6 new GTest cases (22 total).
- gz magnetometer on imu_link (vendored xacro, additive) bridged by
  eskf.launch.py. Measured headless: with <spherical_coordinates> gz uses
  its WMM field in GAUSS (|B| 0.433, 4.0 deg from +x) and ignores the SDF
  <magnetic_field>; noise stddev is in gauss too (0.005 G -> 0.98 deg).
  Heading recovered yaw to 0.000 deg at four poses incl. upside down.
- R grows with the body's tilt LAG behind "up" (gyro high-pass with
  grav_lp_'s time constant): fit sigma^2 = (2.96 deg)^2 + (0.60*lag)^2 on a
  live run, plus a 3-sigma innovation gate with a 5 s lock-out escape.
  Replaying that run's real mag headings: worst yaw error 12.4 -> 7.8 deg.
- run_report.py: mag_heading/mag_err columns and a mag-vs-truth section
  (live terrain squares: std 4.1-4.3 deg, heavy-tailed with tilt).
- yaw_observability.py: magnetometer arms (offline: 2.00 -> 0.61 deg final
  yaw on the square at 2 deg tilt error, worse than GPS alone at 10 deg).

terrain_adapt.py (--adapt)
- Pitch sign FIXED: atan2(-f_x, ...) is REP-103 (+nose-down), not
  +nose-up, so com_shift_x shifted the CoM downhill on every slope and a
  descent became a nose-dive (21:25 fall). Checked on a gz IMU at a known
  8.6 deg nose-up pose. level_pitch was already right (two inversions
  cancelled; verified against CHAMP's RotateY). Every earlier --adapt
  result is invalid.
- Gyro + accel complementary filter (attitude_mode: complementary,
  cf_tau 10 s, bootstrapped). Accel-only read +19 deg on flat ground at
  gait start; offline that transient drops 18.2 -> 4.7 deg. Publishes
  /terrain_adapt/pitch, scored against truth in REPORT.md. Open issue:
  +7 deg nose-up bias while walking, traced to the gyro path.

square_test.py
- Fall height threshold minus the commanded crouch (/body_pose), which
  previously contradicted the adapter by construction (0.165 < 0.18).
- Speed-up ramp only (0 -> 0.25 m/s over 2 s; stops are immediate), and
  steering off a 0.25 s low-passed heading.
- A fall condition pauses and recovers instead of aborting on one sample;
  abort only if it persists 0.5 s or does not settle in 5 s. Stall is now
  the max excursion over the window, so circling a corner is not a stall.

plot_trajectory.py: 2x2 grid with a slip-score panel; the twist panel's
y-range is the central 99 % so ~500 rad/s truth omega_z spikes cannot
flatten it.

Also carries the pre-session GPS-on-by-default work (eskf params/launch,
navsat noise in metres) and a whitespace-only change in state_estimation.h.
Findings and every measurement are in skills.md section 0.

Co-Authored-By: Claude Opus 5.5 (1M context) <noreply@anthropic.com>

File: src/unitree_go2_ros2/unitree_go2_description/urdf/unitree_go2_gazebo.xacro (robot description, xacro)
@@ -101,5 +101,50 @@
             </sensor>
         </gazebo>
-        <!-- GPS / NavSat plugin — simulates u-blox standard GPS (~0.5 m horizontal noise) -->
+        <!-- Magnetometer — VENDORED EDIT (additive), for go2_eskf's heading update.
+             On imu_link, i.e. the SAME frame as the accelerometer, because go2_eskf
+             tilt-compensates it with the low-passed accelerometer as "up" instead of
+             roll/pitch angles (the gz-IMU orientation is unreliable, DESIGN.md §6).
+             Non-rendering, so it adds no GPU load. Bridged by go2_eskf
+             eskf.launch.py use_mag:=true; harmless when nothing subscribes.
+             MEASURED 2026-09-23 (headless gz world, static models at known poses):
+             * Because every Go2 world sets <spherical_coordinates>, gz IGNORES the
+               SDF <magnetic_field> default and computes the field from its WMM tables
+               at the datum, in GAUSS despite the msg field being named field_tesla:
+               |B| = 0.4326, horizontal 0.3096, pointing 4.0 deg from world +x
+               (0.0699 rad) — not the SDF default's 76 deg.
+             * The noise <stddev> is added in those same units, so it is in GAUSS:
+               0.005 G (= 0.5 uT) per axis measured 0.98 deg of heading std.
+             * The tilt-compensated heading recovered the true yaw to 0.000 deg at
+               four poses, including one mounted upside down (roll = pi). -->
+        <xacro:property name="mag_noise_gauss" value="0.005"/>
+        <gazebo reference="imu_link">
+            <sensor name="mag_sensor" type="magnetometer">
+                <always_on>true</always_on>
+                <update_rate>20</update_rate>
+                <topic>imu/mag</topic>
+                <gz_frame_id>imu_link</gz_frame_id>
+                <magnetometer>
+                    <x><noise type="gaussian"><mean>0.0</mean><stddev>${mag_noise_gauss}</stddev></noise></x>
+                    <y><noise type="gaussian"><mean>0.0</mean><stddev>${mag_noise_gauss}</stddev></noise></y>
+                    <z><noise type="gaussian"><mean>0.0</mean><stddev>${mag_noise_gauss}</stddev></noise></z>
+                </magnetometer>
+                <plugin filename="gz-sim-magnetometer-system" name="gz::sim::systems::Magnetometer"/>
+            </sensor>
+        </gazebo>
+        <!-- GPS / NavSat plugin — simulates u-blox standard GPS.
+             VENDORED EDIT (additive): the horizontal position noise is specified
+             in DEGREES, not metres. gz-sensors adds the <stddev> straight onto the
+             latitude/longitude in degrees, so the original <stddev>0.5</stddev>
+             meant ~0.5 deg = ~55 km of scatter, which is why GPS was unusable and
+             switched off by default. Expressed in metres and converted here.
+             The divisor is metres-per-degree at the world datum (lat 30.0444), on
+             the SAME spherical earth model eskf_node's gpsToEnu uses (R=6371 km):
+               1 deg lat = 111195 m,  1 deg lon = 111195*cos(30.0444) = 96269 m.
+             SDF allows only ONE horizontal noise for both axes, so this uses their
+             geometric mean (103459 m/deg); at 0.5 m nominal that lands 0.54 m
+             north/south and 0.46 m east/west. Vertical noise is NOT converted: the
+             altitude field is natively metres, so it was never affected. -->
+        <xacro:property name="gps_noise_m" value="0.5"/>
+        <xacro:property name="gps_m_per_deg" value="103459.0"/>
         <gazebo reference="gps_link">
             <sensor name="navsat_sensor" type="navsat">
@@ -113,5 +158,5 @@
                             <noise type="gaussian">
                                 <mean>0.0</mean>
-                                <stddev>0.5</stddev>
+                                <stddev>${gps_noise_m / gps_m_per_deg}</stddev>
                             </noise>
                         </horizontal>
